Commit message: fix

File: aubo_description/urdf/aubo_i3 (copy).urdf (robot description, URDF)
Before this commit: robot aubo_i3, 15 links, 14 joints
Links:
- link eef_link: geometry collision mesh filename=package://aubo_description/meshes/aubo_i3/collision/eef_sol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; visual mesh filename=package://aubo_description/meshes/aubo_i3/collision/eef_sol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
Joints:
- joint eef_joint: origin xyz=0.0 0.0 0.0 rpy=0 0 0.0 -> xyz=0.005 0.0 0.0 rpy=-2.094395 0 0.0
- joint eelink_finger_joint: origin xyz=0.14600 0.03172 0.08558 rpy=-0.977384364 0 0 -> xyz=0.200 0.024730 0.078580 rpy=-0.977384364 0 0
- joint eelink_palm_joint: origin xyz=0.173930 0.005870 0.059050 rpy=-0.977384364 0 0 -> xyz=0.211430 0.059050 -0.005870 rpy=-0.977384364 0 0
- joint vision_joint: origin xyz=0.117660 -0.036399 0.010216 rpy=-0.967871 0.215096 -0.280483 -> xyz=0.189326 -0.050356 -0.002892 rpy=-0.998538 0.194956 -0.289171

File: aubo_description/urdf/aubo_i3 (old_eefeelink_000).urdf (robot description, URDF)
Before this commit: robot aubo_i3, 15 links, 14 joints
Joints:
- joint eelink_finger_joint: origin xyz=0.14600 0.03172 0.08558 rpy=-0.977384364 0 0 -> xyz=0.200 0.024730 0.078580 rpy=-0.977384364 0 0
- joint eelink_palm_joint: origin xyz=0.173930 0.005870 0.059050 rpy=-0.977384364 0 0 -> xyz=0.211430 0.059050 -0.005870 rpy=-0.977384364 0 0
- joint vision_joint: origin xyz=0.117660 -0.036399 0.010216 rpy=-0.967871 0.215096 -0.280483 -> xyz=0.189326 -0.050356 -0.002892 rpy=-0.998538 0.194956 -0.289171

Commit message: fix bug

File: aubo_description/urdf/aubo_i3 (copy).urdf (robot description, URDF)
Before this commit: robot aubo_i3, 15 links, 14 joints
Links:
- added link finger_rub; visual box size=0.005 0.005 0.005
- link eef_link: geometry collision mesh filename=package://aubo_description/meshes/aubo_i3/collision/eef_sin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; visual mesh filename=package://aubo_description/meshes/aubo_i3/collision/eef_sin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
Joints:
- added joint eelink_finger_rub_joint: type fixed, parent ee_link, child finger_rub, origin xyz=0.18100 0.02826 0.07855 rpy=-1.047197533 0 0
- joint eef_joint: origin xyz=0.005 0.0 0.0 rpy=-2.094395 0 0.0 -> xyz=0.0 0.0 0.0 rpy=0 0 0.0
- joint eelink_finger_joint: origin xyz=0.200 0.024730 0.078580 rpy=-0.977384364 0 0 -> xyz=0.18100 0.038720 0.080580 rpy=-1.047197533 0 0
- joint eelink_palm_joint: origin xyz=0.211430 0.059050 -0.005870 rpy=-0.977384364 0 0 -> xyz=0.173930 0.005870 0.059050 rpy=-1.047197533 0 0
- joint foreArm_joint: limit lower=-0.035 upper=3.1415926 effort=0 velocity=0 -> lower=-0.035 upper=3.036873 effort=0 velocity=0
- joint mounter_joint: origin xyz=0.0 0 0.0 rpy=3.14159 0.0 2.35621 -> xyz=0.0 0 0.0 rpy=3.14159 0.0 4.712389
- joint shoulder_joint: limit lower=-3.1415926 upper=3.1415926 effort=0 velocity=0 -> lower=-3.036873 upper=3.036873 effort=0 velocity=0
- joint vision_joint: origin xyz=0.189326 -0.050356 -0.002892 rpy=-0.998538 0.194956 -0.289171 -> xyz=0.107466 -0.031883 0.005886 rpy=-1.121578 0.168985 -0.313050
- joint world_joint: origin xyz=0.0 -0.658 0.0 rpy=0 0 0.02618 -> xyz=0.0 -0.658 0.0 rpy=0 0 0
- joint wrist2_joint: limit lower=-3.1415926 upper=0.035 effort=0 velocity=0 -> lower=-3.036873 upper=0.035 effort=0 velocity=0
- joint wrist3_joint: limit lower=-1.0472 upper=2.618 effort=0 velocity=0 -> lower=-2.0472 upper=2.618 effort=0 velocity=0

File: aubo_description/urdf/aubo_i3.urdf (robot description, URDF)
Before this commit: robot aubo_i3, 16 links, 15 joints
Joints:
- joint eelink_finger_joint: origin xyz=0.17600 0.038720 0.080580 rpy=-0.977384364 0 0 -> xyz=0.181000 0.032720 0.086580 rpy=-1.047197533 0 0
- joint eelink_finger_rub_joint: origin xyz=0.166500 0.02826 0.07855 rpy=-0.977384364 0 0 -> xyz=0.181000 0.025960 0.084050 rpy=-1.047197533 0 0
- joint eelink_palm_joint: origin xyz=0.173930 0.005870 0.059050 rpy=-0.977384364 0 0 -> xyz=0.173930 0.005870 0.059050 rpy=-1.047197533 0 0
- joint vision_joint: origin xyz=0.107466 -0.031883 0.005886 rpy=-1.121578 0.168985 -0.313050 -> xyz=0.108847 -0.030902 0.008042 rpy=-1.130905 0.171703 -0.317177

Commit message: rebase master

File: aubo_description/urdf/aubo_i3 (copy).urdf (robot description, URDF)
Before this commit: robot aubo_i3, 16 links, 15 joints
Joints:
- joint eelink_finger_joint: origin xyz=0.181000 0.032720 0.086580 rpy=-1.047197533 0 0 -> xyz=0.18100 0.038720 0.080580 rpy=-1.047197533 0 0
- joint eelink_finger_rub_joint: origin xyz=0.181000 0.025960 0.084050 rpy=-1.047197533 0 0 -> xyz=0.18100 0.02826 0.07855 rpy=-1.047197533 0 0
- joint foreArm_joint: limit lower=-0.035 upper=2.6179939 effort=0 velocity=0 -> lower=-0.035 upper=3.036873 effort=0 velocity=0
- joint vision_joint: origin xyz=0.108847 -0.030902 0.008042 rpy=-1.130905 0.171703 -0.317177 -> xyz=0.107466 -0.031883 0.005886 rpy=-1.121578 0.168985 -0.313050

File: aubo_description/urdf/aubo_i3 (old_eefeelink_000).urdf (robot description, URDF)
Before this commit: robot aubo_i3, 16 links, 15 joints
Links:
- removed link finger_rub
Joints:
- removed joint eelink_finger_rub_joint
- joint eelink_finger_joint: origin xyz=0.181000 0.032720 0.086580 rpy=-1.047197533 0 0 -> xyz=0.200 0.024730 0.078580 rpy=-0.977384364 0 0
- joint eelink_palm_joint: origin xyz=0.173930 0.005870 0.059050 rpy=-1.047197533 0 0 -> xyz=0.211430 0.059050 -0.005870 rpy=-0.977384364 0 0
- joint foreArm_joint: limit lower=-0.035 upper=2.6179939 effort=0 velocity=0 -> lower=-0.035 upper=3.1415926 effort=0 velocity=0
- joint mounter_joint: origin xyz=0.0 0 0.0 rpy=3.14159 0.0 4.712389 -> xyz=0.0 0 0.0 rpy=3.14159 0.0 2.35621
- joint shoulder_joint: limit lower=-3.036873 upper=3.036873 effort=0 velocity=0 -> lower=-3.1415926 upper=3.1415926 effort=0 velocity=0
- joint vision_joint: origin xyz=0.108847 -0.030902 0.008042 rpy=-1.130905 0.171703 -0.317177 -> xyz=0.189326 -0.050356 -0.002892 rpy=-0.998538 0.194956 -0.289171
- joint world_joint: origin xyz=0.0 -0.658 0.0 rpy=0 0 0 -> xyz=0.0 -0.658 0.0 rpy=0 0 0.02618
- joint wrist2_joint: limit lower=-3.036873 upper=0.035 effort=0 velocity=0 -> lower=-3.1415926 upper=0.035 effort=0 velocity=0
- joint wrist3_joint: limit lower=-2.0472 upper=2.618 effort=0 velocity=0 -> lower=-1.0472 upper=2.618 effort=0 velocity=0

File: aubo_gazebo/urdf/aubo_i3.xacro (robot description, xacro)
@@ -234,5 +234,5 @@
     <parent link="foreArm_Link" />
     <child link="wrist1_Link" />
-    <axis xyz="0 0 1" />
+    <axis xyz="0 0 -1" />
     <limit lower="-3.05" upper="3.05" effort="300" velocity="100" />
   </joint>
@@ -292,5 +292,5 @@
     <parent link="wrist2_Link" />
     <child link="wrist3_Link" />
-    <axis xyz="0 0 1" />
+    <axis xyz="0 0 -1" />
     <limit lower="-3.05" upper="3.05" effort="300" velocity="100" />
   </joint>
@@ -300,57 +300,53 @@
   <joint name="world_joint" type="fixed">
     <origin xyz="0 0 0.05" rpy="0 0 0" />
-    <!--<origin xyz="0 0 0" rpy="0 0 0" />-->
     <parent link="world" />
     <child link = "pedestal_Link" />
     <origin xyz="0.0 0.0 0.0" rpy="0.0 0.0 0.0" />
   </joint>
-<!--/////////////////////////////// pedestal_Link ////////////////////////////////////-->
- <link name="pedestal_Link">
-   <visual>
-    <geometry>
-      <box size="1.0 1.0 0.1" />
-<!--      <box size="0.0 0.0 0.0" />-->
-    </geometry>
-    <material name="">
-       <color rgba="0.96 0.96 0.96 1" />
-    </material>
-   </visual>
-  </link>
-<!--/////////////////////////////// pedestal_JOINIT ////////////////////////////////////-->
+ <!--/////////////////////////////// pedestal_Link ////////////////////////////////////-->
+  <link name="pedestal_Link">
+    <visual>
+     <geometry>
+       <box size="1.5 1.5 0.1" />
+     </geometry>
+     <material name="">
+        <color rgba="0.96 0.96 0.96 1" />
+     </material>
+    </visual>
+   </link>
+ <!--/////////////////////////////// pedestal_JOINIT ////////////////////////////////////-->
 <joint name="pedestal_joint" type="fixed">
-   <origin xyz="0 0 0.051" rpy="0 0 0" />
-   <!--<origin xyz="0 0 0" rpy="0 0 0" />-->
-   <parent link="pedestal_Link" />
-   <child link = "base_link" />
-<!--   <child link = "pedestal_Link" />-->
-   <origin xyz="0.0 0.0 0.0" rpy="0.0 0.0 0.0" />
- </joint>
- <!-- /////////////////////////////////   gazebo color   ////////////////////////////////////// -->
- <gazebo reference="pedestal_Link">
-    <material>Gazebo/Grey</material>
- </gazebo>
- <!--////////////////////////////////// Transmissions for ROS Control //////////////////////////-->
- <xacro:macro name="aubo_arm_transmission" params="joint_name">
-     <transmission name="${joint_name}_trans">
-       <type>transmission_interface/SimpleTransmission</type>
-       <joint name="${joint_name}">
-         <hardwareInterface>hardware_interface/PositionJointInterface</hardwareInterface>
-       </joint>
-       <actuator name="${joint_name}_motor">
-         <mechanicalReduction>1</mechanicalReduction>
-       </actuator>
-     </transmission>
- </xacro:macro>
- <xacro:aubo_arm_transmission joint_name="shoulder_joint"/>
- <xacro:aubo_arm_transmission joint_name="upperArm_joint"/>
- <xacro:aubo_arm_transmission joint_name="foreArm_joint"/>
- <xacro:aubo_arm_transmission joint_name="wrist1_joint"/>
- <xacro:aubo_arm_transmission joint_name="wrist2_joint"/>
- <xacro:aubo_arm_transmission joint_name="wrist3_joint"/>
- <!-- ros_control plugin -->
- <gazebo>
-     <plugin name="gazebo_ros_control" filename="libgazebo_ros_control.so">
-         <robotNamespace>/aubo_i3</robotNamespace>
-     </plugin>
- </gazebo>
+    <origin xyz="0 0 0.051" rpy="0 0 0" />
+    <parent link="pedestal_Link" />
+    <child link = "base_link" />
+    <origin xyz="0.0 0.0 0.0" rpy="0.0 0.0 0.0" />
+  </joint>
+  <!-- /////////////////////////////////   gazebo color   ////////////////////////////////////// -->
+  <gazebo reference="pedestal_Link">
+     <material>Gazebo/Grey</material>
+  </gazebo>
+  <!--////////////////////////////////// Transmissions for ROS Control //////////////////////////-->
+  <xacro:macro name="aubo_arm_transmission" params="joint_name">
+      <transmission name="${joint_name}_trans">
+        <type>transmission_interface/SimpleTransmission</type>
+        <joint name="${joint_name}">
+          <hardwareInterface>hardware_interface/PositionJointInterface</hardwareInterface>
+        </joint>
+        <actuator name="${joint_name}_motor">
+          <mechanicalReduction>1</mechanicalReduction>
+        </actuator>
+      </transmission>
+  </xacro:macro>
+  <xacro:aubo_arm_transmission joint_name="shoulder_joint"/>
+  <xacro:aubo_arm_transmission joint_name="upperArm_joint"/>
+  <xacro:aubo_arm_transmission joint_name="foreArm_joint"/>
+  <xacro:aubo_arm_transmission joint_name="wrist1_joint"/>
+  <xacro:aubo_arm_transmission joint_name="wrist2_joint"/>
+  <xacro:aubo_arm_transmission joint_name="wrist3_joint"/>
+  <!-- ros_control plugin -->
+  <gazebo>
+      <plugin name="gazebo_ros_control" filename="libgazebo_ros_control.so">
+          <robotNamespace>/aubo_i3</robotNamespace>
+      </plugin>
+  </gazebo>
 </robot>
