Commit message: add a msg, armCmdCallback, movej movep

File: aubo_description/urdf/aubo_i3.urdf (robot description, URDF)
Before this commit: robot aubo_i3, 15 links, 14 joints
Links:
- link eef_link: mass 0.1 -> None
- link mounter: mass 0.1 -> None
Joints:
- joint eelink_palm_joint: origin xyz=0.188930 0.005870 0.059050 rpy=0.59341 0 0 -> xyz=0.21175 0.003316 0.00216 rpy=0.59341 0 0
- joint foreArm_joint: limit lower=-2.96705 upper=-0.08726 effort=0 velocity=0 -> lower=-3.05 upper=3.05 effort=0 velocity=0
- joint mounter_joint: origin xyz=0.0 0 0.0 rpy=3.14159 0.0 5.49780 -> xyz=0.0 0 0.0 rpy=3.14159 0.0 2.35621
- joint shoulder_joint: limit lower=-5.41052 upper=1.74532 effort=0 velocity=0 -> lower=-3.05 upper=3.05 effort=0 velocity=0
- joint upperArm_joint: limit lower=-3.31612 upper=-0.78539 effort=0 velocity=0 -> lower=-3.05 upper=3.05 effort=0 velocity=0
- joint vision_joint: origin xyz=-0.172481 0.102860 -0.090900 rpy=0.105282 -0.048103 -0.107558 -> xyz=0.14337 -0.03420 0.00467 rpy=-0.905282 0.248103 -0.307558
- joint wrist1_joint: axis 0 0 -1 -> 0 0 1; limit lower=-4.71239 upper=0.0 effort=0 velocity=0 -> lower=-3.05 upper=3.05 effort=0 velocity=0
- joint wrist2_joint: limit lower=-1.57080 upper=0.0 effort=0 velocity=0 -> lower=-3.05 upper=3.05 effort=0 velocity=0
- joint wrist3_joint: axis 0 0 -1 -> 0 0 1; limit lower=-1.29154 upper=2.96705 effort=0 velocity=0 -> lower=-3.05 upper=3.05 effort=0 velocity=0

File: aubo_description/urdf/aubo_i3.urdf.xacro (robot description, xacro)
@@ -206,31 +206,7 @@
   <link name="world" />
   <joint name="world_joint" type="fixed">
-    <parent link="world"/>
-    <child link="mounter"/>
-    <origin xyz="0.0 -0.658 0.0" rpy="0 0 0"/>
-  </joint>
-  <link name="mounter">
-    <visual>
-      <geometry>
-        <mesh filename="package://aubo_description/meshes/aubo_i3/collision/mounter_front_new.stl"/>
-      </geometry>
-      <material name="LightGrey">
-        <color rgba="0.7 0.7 0.7 1.0"/>
-      </material>
-    </visual>
-    <collision>
-      <geometry>
-        <mesh filename="package://aubo_description/meshes/aubo_i3/collision/mounter_front_new.stl"/>
-      </geometry>
-    </collision>
-    <inertial>
-      <mass value="0.1"/>
-      <inertia ixx="0.00003" iyy="0.00003" izz="0.00003" ixy="0.0" ixz="0.0" iyz="0.0"/>
-    </inertial>
-  </link>
-  <joint name="mounter_joint" type="fixed">
-    <parent link="mounter"/>
-    <child link="base_link"/>
-    <origin xyz="0.0 0 0.0" rpy="3.14159 0.0 5.49780"/>
+    <parent link="world" />
+    <child link = "mounter" />
+    <origin xyz="0.0 -0.658 0.0" rpy="0.0 0.0 0.0" />
   </joint>
 </robot>

Commit message: modify some error

File: aubo_description/urdf/aubo_i3.urdf (robot description, URDF)
Before this commit: robot aubo_i3, 15 links, 14 joints
Joints:
- joint eef_joint: origin xyz=0.0 0.0 0.0 rpy=0 0 0.0 -> xyz=0.0 0.0 0.0 rpy=-2.094395 0 0.0
- joint eelink_finger_joint: origin xyz=0.181500 -0.071350 0.028340 rpy=0.59341 0 0 -> xyz=0.189280 -0.071350 0.028340 rpy=-0.785398 0 0
- joint foreArm_joint: limit lower=-3.05 upper=3.05 effort=0 velocity=0 -> lower=-3.1416 upper=3.1416 effort=0 velocity=0
- joint shoulder_joint: limit lower=-3.05 upper=3.05 effort=0 velocity=0 -> lower=-3.1416 upper=3.1416 effort=0 velocity=0
- joint upperArm_joint: limit lower=-3.05 upper=3.05 effort=0 velocity=0 -> lower=-3.1416 upper=3.1416 effort=0 velocity=0
- joint wrist1_joint: limit lower=-3.05 upper=3.05 effort=0 velocity=0 -> lower=-3.1416 upper=3.1416 effort=0 velocity=0
- joint wrist2_joint: limit lower=-3.05 upper=3.05 effort=0 velocity=0 -> lower=-3.1416 upper=3.1416 effort=0 velocity=0
- joint wrist3_joint: limit lower=-3.05 upper=3.05 effort=0 velocity=0 -> lower=-3.1416 upper=3.1416 effort=0 velocity=0

File: aubo_description/urdf/aubo_i3_robot.urdf.xacro (robot description, xacro)
@@ -7,10 +7,16 @@
   <xacro:include filename="$(find aubo_description)/urdf/aubo_i3.urdf.xacro" />
   <!-- arm -->
-  <xacro:aubo_i5L_robot prefix="" joint_limited="false"/>
+  <xacro:aubo_i3_robot prefix="" joint_limited="false"/>
   <link name="world" />
   <joint name="world_joint" type="fixed">
     <parent link="world" />
+    <child link = "mounter" />
+     <origin xyz="0.0 -0.658 0.0" rpy="0 0 0.02618" />
+  </joint>
+  <link name="mounter" />
+  <joint name="mounter_joint" type="fixed">
+    <parent link="mounter" />
     <child link = "base_link" />
-    <origin xyz="0.0 0.0 0.0" rpy="0.0 0.0 0.0" />
+    <origin xyz="0.0 0 0.0" rpy="3.14159 0.0 2.35621"/>
   </joint>
 </robot>

Commit message: fix bug

File: aubo_description/urdf/aubo_i3.urdf (robot description, URDF)
Before this commit: robot aubo_i3, 15 links, 14 joints
Joints:
- joint eelink_finger_joint: origin xyz=0.189280 -0.071350 0.028340 rpy=-0.785398 0 0 -> xyz=0.227500 0.028080 0.071870 rpy=0 0 0
- joint eelink_palm_joint: origin xyz=0.21175 0.003316 0.00216 rpy=0.59341 0 0 -> xyz=0.211430 0.059050 -0.005870 rpy=-0.977384381 0 0
- joint foreArm_joint: limit lower=-3.1416 upper=3.1416 effort=0 velocity=0 -> lower=-2.094395102 upper=3.1415926 effort=0 velocity=0
- joint shoulder_joint: limit lower=-3.1416 upper=3.1416 effort=0 velocity=0 -> lower=-3.1415926 upper=3.1415926 effort=0 velocity=0
- joint upperArm_joint: limit lower=-3.1416 upper=3.1416 effort=0 velocity=0 -> lower=-2.094395102 upper=2.094395102 effort=0 velocity=0
- joint vision_joint: origin xyz=0.14337 -0.03420 0.00467 rpy=-0.905282 0.248103 -0.307558 -> xyz=0.192777 -0.038643 -0.000208 rpy=-1.039315 0.180144 -0.295751
- joint wrist1_joint: limit lower=-3.1416 upper=3.1416 effort=0 velocity=0 -> lower=-1.396263402 upper=1.396263402 effort=0 velocity=0
- joint wrist3_joint: limit lower=-3.1416 upper=3.1416 effort=0 velocity=0 -> lower=-3.1415926 upper=3.1415926 effort=0 velocity=0

Commit message: modify something

File: aubo_description/urdf/aubo_i3.urdf (robot description, URDF)
Before this commit: robot aubo_i3, 15 links, 14 joints
Joints:
- joint eelink_finger_joint: origin xyz=0.227500 0.028080 0.071870 rpy=0 0 0 -> xyz=0.227500 0.028080 0.071870 rpy=-0.977384364 0 0
- joint foreArm_joint: limit lower=-2.094395102 upper=3.1415926 effort=0 velocity=0 -> lower=-0.035 upper=3.1415926 effort=0 velocity=0
- joint upperArm_joint: limit lower=-2.094395102 upper=2.094395102 effort=0 velocity=0 -> lower=-2.0944 upper=2.0944 effort=0 velocity=0
- joint wrist1_joint: limit lower=-1.396263402 upper=1.396263402 effort=0 velocity=0 -> lower=-1.3963 upper=1.3963 effort=0 velocity=0
- joint wrist2_joint: limit lower=-3.1416 upper=3.1416 effort=0 velocity=0 -> lower=-3.1415926 upper=0.035 effort=0 velocity=0
- joint wrist3_joint: limit lower=-3.1415926 upper=3.1415926 effort=0 velocity=0 -> lower=-1.0472 upper=2.618 effort=0 velocity=0

Commit message: 1

File: aubo_description/urdf/aubo_i3.urdf (robot description, URDF)
Before this commit: robot aubo_i3, 15 links, 14 joints
Joints:
- joint eelink_palm_joint: origin xyz=0.211430 0.059050 -0.005870 rpy=-0.977384381 0 0 -> xyz=0.231430 0.059050 -0.005870 rpy=-0.977384381 0 0

Commit message: fix

File: aubo_description/urdf/aubo_i3.urdf (robot description, URDF)
Before this commit: robot aubo_i3, 15 links, 14 joints
Links:
- link eef_link: geometry collision mesh filename=package://aubo_description/meshes/aubo_i3/collision/eef_sol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; visual mesh filename=package://aubo_description/meshes/aubo_i3/collision/eef_sol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
Joints:
- joint eef_joint: origin xyz=0.0 0.0 0.0 rpy=-2.094395 0 0.0 -> xyz=0.005 0.0 0.0 rpy=-2.094395 0 0.0
- joint eelink_finger_joint: origin xyz=0.227500 0.028080 0.071870 rpy=-0.977384364 0 0 -> xyz=0.247330 0.024730 0.078580 rpy=-0.977384364 0 0
- joint eelink_palm_joint: origin xyz=0.231430 0.059050 -0.005870 rpy=-0.977384381 0 0 -> xyz=0.211430 0.059050 -0.005870 rpy=-0.977384364 0 0
- joint vision_joint: origin xyz=0.192777 -0.038643 -0.000208 rpy=-1.039315 0.180144 -0.295751 -> xyz=0.189326 -0.050356 -0.002892 rpy=-0.998538 0.194956 -0.289171

Commit message: fix bug

File: aubo_description/urdf/aubo_i3.urdf (robot description, URDF)
Before this commit: robot aubo_i3, 15 links, 14 joints
Joints:
- joint eelink_finger_joint: origin xyz=0.14600 0.03172 0.08558 rpy=-0.977384364 0 0 -> xyz=0.161000 0.029720 0.075580 rpy=-0.977384364 0 0
- joint mounter_joint: origin xyz=0.0 0 0.0 rpy=3.14159 0.0 2.35621 -> xyz=0.0 0 0.0 rpy=3.14159 0.0 3.14159
- joint vision_joint: origin xyz=0.117660 -0.036399 0.010216 rpy=-0.967871 0.215096 -0.280483 -> xyz=0.118007 -0.035189 0.012310 rpy=-1.016933 0.220174 -0.290849
- joint world_joint: origin xyz=0.0 -0.658 0.0 rpy=0 0 0.02618 -> xyz=0.0 -0.658 0.0 rpy=0 0 0

Commit message: add finger rub

File: aubo_description/urdf/aubo_i3.urdf (robot description, URDF)
Before this commit: robot aubo_i3, 15 links, 14 joints
Links:
- added link finger_rub; visual box size=0.005 0.005 0.005
Joints:
- added joint eelink_finger_rub_joint: type fixed, parent ee_link, child finger_rub, origin xyz=0.166500 0.01926 0.07155 rpy=-0.977384364 0 0

Commit message: fix bug

File: aubo_description/urdf/aubo_i3.urdf (robot description, URDF)
Before this commit: robot aubo_i3, 15 links, 14 joints
Joints:
- joint eelink_finger_joint: origin xyz=0.166500 0.026720 0.076580 rpy=-0.977384364 0 0 -> xyz=0.17600 0.033720 0.083580 rpy=-0.977384364 0 0
- joint vision_joint: origin xyz=0.108242 -0.031091 0.010288 rpy=-1.048239 0.187654 -0.300688 -> xyz=0.107466 -0.031883 0.005886 rpy=-1.121578 0.168985 -0.313050

Commit message: fix bug

File: aubo_description/urdf/aubo_i3.urdf (robot description, URDF)
Before this commit: robot aubo_i3, 16 links, 15 joints
Joints:
- joint eelink_finger_rub_joint: origin xyz=0.166500 0.01926 0.07155 rpy=-0.977384364 0 0 -> xyz=0.166500 0.02626 0.07855 rpy=-0.977384364 0 0

Commit message: fix bug

File: aubo_description/urdf/aubo_i3.urdf (robot description, URDF)
Before this commit: robot aubo_i3, 16 links, 15 joints
Joints:
- joint eelink_finger_joint: origin xyz=0.17600 0.033720 0.083580 rpy=-0.977384364 0 0 -> xyz=0.17600 0.038720 0.080580 rpy=-0.977384364 0 0
- joint eelink_finger_rub_joint: origin xyz=0.166500 0.02626 0.07855 rpy=-0.977384364 0 0 -> xyz=0.166500 0.02826 0.07855 rpy=-0.977384364 0 0

Commit message: fix bug

File: aubo_description/urdf/aubo_i3.urdf (robot description, URDF)
Before this commit: robot aubo_i3, 16 links, 15 joints
Joints:
- joint foreArm_joint: limit lower=-0.035 upper=3.036873 effort=0 velocity=0 -> lower=-0.035 upper=2.6179939 effort=0 velocity=0

Commit message: Add emma basic communication and control

File: aubo_description/urdf/aubo_i3.urdf (robot description, URDF)
Before this commit: robot aubo_i3, 8 links, 7 joints
Links:
- added link camera_link; visual box size=0.005 0.005 0.005
- added link ee_link; visual box size=0.005 0.005 0.005
- added link eef_link; collision mesh filename=package://aubo_description/meshes/aubo_i3/collision/eef_sin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; visual mesh filename=package://aubo_description/meshes/aubo_i3/collision/eef_sin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
- added link finger; visual box size=0.005 0.005 0.005
- added link finger_rub; visual box size=0.005 0.005 0.005
- added link mounter; collision mesh filename=package://aubo_description/meshes/aubo_i3/collision/mounter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; visual mesh filename=package://aubo_description/meshes/aubo_i3/collision/mounter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
- added link palm; visual box size=0.005 0.005 0.005
- added link tool0
Joints:
- added joint ee_fixed_joint: type fixed, parent wrist3_Link, child ee_link, origin xyz=0.0 0.0 0.0 rpy=0.0 -1.57079 0
- added joint eef_joint: type fixed, parent ee_link, child eef_link, origin xyz=0.0 0.0 0.0 rpy=0 0 0.0
- added joint eelink_finger_joint: type fixed, parent ee_link, child finger, origin xyz=0.181000 0.032720 0.086580 rpy=-1.047197533 0 0
- added joint eelink_finger_rub_joint: type fixed, parent ee_link, child finger_rub, origin xyz=0.181000 0.025960 0.084050 rpy=-1.047197533 0 0
- added joint eelink_palm_joint: type fixed, parent ee_link, child palm, origin xyz=0.173930 0.005870 0.059050 rpy=-1.047197533 0 0
- added joint mounter_joint: type fixed, parent mounter, child base_link, origin xyz=0.0 0 0.0 rpy=3.14159 0.0 4.712389
- added joint vision_joint: type fixed, parent ee_link, child camera_link, origin xyz=0.108847 -0.030902 0.008042 rpy=-1.130905 0.171703 -0.317177
- added joint wrist3_Link-tool0_fixed_joint: type fixed, parent wrist3_Link, child tool0, origin xyz=0 0 0 rpy=-1.57079 0 0
- joint foreArm_joint: limit lower=-3.05 upper=3.05 effort=0 velocity=0 -> lower=-0.035 upper=2.6179939 effort=0 velocity=0
- joint shoulder_joint: limit lower=-3.05 upper=3.05 effort=0 velocity=0 -> lower=-3.036873 upper=3.036873 effort=0 velocity=0
- joint upperArm_joint: limit lower=-3.05 upper=3.05 effort=0 velocity=0 -> lower=-2.0944 upper=2.0944 effort=0 velocity=0
- joint world_joint: child base_link -> mounter; origin xyz=0.0 0.0 0.0 rpy=0.0 0.0 0.0 -> xyz=0.0 -0.658 0.0 rpy=0 0 0
- joint wrist1_joint: axis 0 0 -1 -> 0 0 1; limit lower=-3.05 upper=3.05 effort=0 velocity=0 -> lower=-1.3963 upper=1.3963 effort=0 velocity=0
- joint wrist2_joint: limit lower=-3.05 upper=3.05 effort=0 velocity=0 -> lower=-3.036873 upper=0.035 effort=0 velocity=0
- joint wrist3_joint: axis 0 0 -1 -> 0 0 1; limit lower=-3.05 upper=3.05 effort=0 velocity=0 -> lower=-2.0472 upper=2.618 effort=0 velocity=0
